Commit message: DONATELLO YA SE MUEVE: * Se han fijado las articulaciones "axle" para que no vuelque el robot (estudiar esto más adelante) * En gazebo.xacro se eliminan los "axle" del plugin (si no, da error) * Se ha subido el peso del base_link

File: urdf/donatello.urdf.xacro (robot description, xacro)
@@ -36,7 +36,7 @@
         </collision>
         <inertial>
-            <mass value="1.0"/>
-            <origin xyz="0 0 0"/>
-            <inertia ixx="0.083" ixy="0.0" ixz="0.0" iyy="0.021" iyz="0.0" izz="0.1"/>
+            <mass value="20.0"/>
+            <origin xyz="0 0 0"/>
+            <inertia ixx="0.3" ixy="0.0" ixz="0.0" iyy="0.3" iyz="0.0" izz="0.3"/>
         </inertial>
     </link>
@@ -164,4 +164,5 @@
         <origin xyz="0 0 0" rpy="0 0 0"/>
     </joint>
+    <!--
     <joint name="rear_axle_joint" type="continuous">
         <parent link="base_link"/>
@@ -181,4 +182,20 @@
         <origin xyz="0.3 ${-(0.3+prism_width/2)} -0.15" rpy="0 0 0"/>
         <axis xyz="0 1 0"/>
+    </joint>
+    -->
+    <joint name="rear_axle_joint" type="fixed">
+        <parent link="base_link"/>
+        <child link="rear_axle_link"/>
+        <origin xyz="${-base_x/2} 0 -0.15" rpy="0 0 0"/>
+    </joint>
+    <joint name="front_left_axle_joint" type="fixed">
+        <parent link="base_link"/>
+        <child link="front_left_axle_link"/>
+        <origin xyz="0.3 ${0.3+prism_width/2} -0.15" rpy="0 0 0"/>
+    </joint>
+    <joint name="front_right_axle_joint" type="fixed">
+        <parent link="base_link"/>
+        <child link="front_right_axle_link"/>
+        <origin xyz="0.3 ${-(0.3+prism_width/2)} -0.15" rpy="0 0 0"/>
     </joint>
     <xacro:wheel prefix="back_left_wheel" parent="rear_axle_link" x="${-rear_cyl_l-prism_width/2}" y="${rear_width/2+prism_width+0.1/2}" z="${-axle_height}" width="${wheel_width}" radius="${wheel_radius}" roll="${-pi/2}"/>

File: urdf/gazebo.xacro (robot description, xacro)
@@ -1,7 +1,14 @@
 <?xml version="1.0"?>
 <robot xmlns:xacro="http://www.ros.org/wiki/xacro">
+    <!--
     <gazebo>
         <plugin name="joint_state_publisher" filename="libgazebo_ros_joint_state_publisher.so">
             <jointName>rear_axle_joint, front_left_axle_joint, front_right_axle_joint, back_left_wheel_joint, back_right_wheel_joint, center_left_wheel_joint, center_right_wheel_joint, front_left_wheel_joint, front_right_wheel_joint</jointName>
+            <update_rate>20.0</update_rate>
+        </plugin>
+    </gazebo>-->
+    <gazebo>
+        <plugin name="joint_state_publisher" filename="libgazebo_ros_joint_state_publisher.so">
+            <jointName>back_left_wheel_joint, back_right_wheel_joint, center_left_wheel_joint, center_right_wheel_joint, front_left_wheel_joint, front_right_wheel_joint</jointName>
             <update_rate>20.0</update_rate>
         </plugin>
