Commit message: added variables for sizes

File: urdf/donatello.urdf (robot description, URDF)
Before this commit: robot donatello, 11 links, 10 joints
Links:
- link base_link: geometry collision box size=1.0 0.6 0.4; visual box size=1.0 0.6 0.4

File: urdf/donatello.urdf.xacro (robot description, xacro)
@@ -7,4 +7,16 @@
     <xacro:property name="pi" value="3.1415926"/>
     <xacro:property name="sqrt_2" value="1.41421356"/>
+    <!-- SIZES -->
+    <xacro:property name="prism_width" value="0.05"/>
+    <xacro:property name="base_x" value="1.0"/>
+    <xacro:property name="base_y" value="0.6"/>
+    <xacro:property name="base_z" value="0.4"/>
+    <xacro:property name="rear_cyl_l" value="0.05"/>
+    <xacro:property name="rear_cyl_r" value="0.025"/>
+    <xacro:property name="rear_width" value="0.6"/>
+    <xacro:property name="axle_height" value="0.4"/>
+    <xacro:property name="wheel_width" value="0.1"/>
+    <xacro:property name="wheel_radius" value="0.1"/>
+    <!-- INERTIA -->
     <!-- LINKS -->
     <link name="dummy_link">
@@ -13,10 +25,10 @@
         <visual>
             <geometry>
-                <box size="1 0.6 0.4"/>
+                <box size="${base_x} ${base_y} ${base_z}"/>
             </geometry>
         </visual>
         <collision>
             <geometry>
-                <box size="1 0.6 0.4"/>
+                <box size="${base_x} ${base_y} ${base_z}"/>
             </geometry>
         </collision>
@@ -30,49 +42,49 @@
         <visual>
             <geometry>
-                <cylinder length="0.05" radius="0.025"/>
+                <cylinder length="${rear_cyl_l}" radius="${rear_cyl_r}"/>
             </geometry>
-            <origin xyz="${-0.05/2} 0 0" rpy="0 ${-pi/2} 0"/>
+            <origin xyz="${-rear_cyl_l/2} 0 0" rpy="0 ${-pi/2} 0"/>
         </visual>
         <visual>
             <geometry>
-                <box size="0.05 0.6 0.05"/>
+                <box size="${prism_width} ${rear_width} ${prism_width}"/>
             </geometry>
-            <origin xyz="${-0.05-0.05/2} 0 0" rpy="0 0 0"/>
+            <origin xyz="${-rear_cyl_l-prism_width/2} 0 0" rpy="0 0 0"/>
         </visual>
         <visual>
             <geometry>
-                <box size="0.05 0.05 0.4"/>
+                <box size="${prism_width} ${prism_width} ${axle_height}"/>
             </geometry>
-            <origin xyz="${-0.05-0.05/2} ${0.6/2+0.05/2} ${-0.4/2+0.05/2}" rpy="0 0 0"/>
+            <origin xyz="${-rear_cyl_l-prism_width/2} ${rear_width/2+prism_width/2} ${-axle_height/2+prism_width/2}" rpy="0 0 0"/>
         </visual>
         <visual>
             <geometry>
-                <box size="0.05 0.05 0.4"/>
+                <box size="${prism_width} ${prism_width} ${axle_height}"/>
             </geometry>
-            <origin xyz="${-0.05-0.05/2} ${-(0.6/2+0.05/2)} ${-0.4/2+0.05/2}" rpy="0 0 0"/>
+            <origin xyz="${-rear_cyl_l-prism_width/2} ${-(rear_width/2+prism_width/2)} ${-axle_height/2+prism_width/2}" rpy="0 0 0"/>
         </visual>
         <collision>
             <geometry>
-                <cylinder length="0.05" radius="0.025"/>
+                <cylinder length="${rear_cyl_l}" radius="${rear_cyl_r}"/>
             </geometry>
-            <origin xyz="0 0 0" rpy="0 ${-pi/2} 0"/>
+            <origin xyz="${-rear_cyl_l/2} 0 0" rpy="0 ${-pi/2} 0"/>
         </collision>
         <collision>
             <geometry>
-                <box size="0.05 0.6 0.05"/>
+                <box size="${prism_width} ${rear_width} ${prism_width}"/>
             </geometry>
-            <origin xyz="${-0.05-0.05/2} 0 0" rpy="0 0 0"/>
+            <origin xyz="${-rear_cyl_l-prism_width/2} 0 0" rpy="0 0 0"/>
         </collision>
         <collision>
             <geometry>
-                <box size="0.05 0.05 0.4"/>
+                <box size="${prism_width} ${prism_width} ${axle_height}"/>
             </geometry>
-            <origin xyz="${-0.05-0.05/2} ${0.6/2+0.05/2} ${-0.4/2+0.05/2}" rpy="0 0 0"/>
+            <origin xyz="${-rear_cyl_l-prism_width/2} ${rear_width/2+prism_width/2} ${-axle_height/2+prism_width/2}" rpy="0 0 0"/>
         </collision>
         <collision>
             <geometry>
-                <box size="0.05 0.05 0.4"/>
+                <box size="${prism_width} ${prism_width} ${axle_height}"/>
             </geometry>
-            <origin xyz="${-0.05-0.05/2} ${-(0.6/2+0.05/2)} ${-0.4/2+0.05/2}" rpy="0 0 0"/>
+            <origin xyz="${-rear_cyl_l-prism_width/2} ${-(rear_width/2+prism_width/2)} ${-axle_height/2+prism_width/2}" rpy="0 0 0"/>
         </collision>
         <inertial>
@@ -85,25 +97,25 @@
         <visual>
             <geometry>
-                <box size="0.05 0.05 ${sqrt_2*0.4}"/>
+                <box size="${prism_width} ${prism_width} ${sqrt_2*base_z}"/>
             </geometry>
-            <origin xyz="${-0.4/2} 0 ${-0.4/2}" rpy="0 ${pi/4} 0"/>
+            <origin xyz="${-axle_height/2} 0 ${-axle_height/2}" rpy="0 ${pi/4} 0"/>
         </visual>
         <visual>
             <geometry>
-                <box size="0.05 0.05 ${sqrt_2*0.4}"/>
+                <box size="${prism_width} ${prism_width} ${sqrt_2*base_z}"/>
             </geometry>
-            <origin xyz="${0.4/2} 0 ${-0.4/2}" rpy="0 ${-pi/4} 0"/>
+            <origin xyz="${axle_height/2} 0 ${-axle_height/2}" rpy="0 ${-pi/4} 0"/>
         </visual>
         <collision>
             <geometry>
-                <box size="0.05 0.05 ${sqrt_2*0.4}"/>
+                <box size="${prism_width} ${prism_width} ${sqrt_2*base_z}"/>
             </geometry>
-            <origin xyz="${-0.4/2} 0 ${-0.4/2}" rpy="0 ${pi/4} 0"/>
+            <origin xyz="${-axle_height/2} 0 ${-axle_height/2}" rpy="0 ${pi/4} 0"/>
         </collision>
         <collision>
             <geometry>
-                <box size="0.05 0.05 ${sqrt_2*0.4}"/>
+                <box size="${prism_width} ${prism_width} ${sqrt_2*base_z}"/>
             </geometry>
-            <origin xyz="${0.4/2} 0 ${-0.4/2}" rpy="0 ${-pi/4} 0"/>
+            <origin xyz="${axle_height/2} 0 ${-axle_height/2}" rpy="0 ${-pi/4} 0"/>
         </collision>
         <inertial>
@@ -116,25 +128,25 @@
         <visual>
             <geometry>
-                <box size="0.05 0.05 ${sqrt_2*0.4}"/>
+                <box size="${prism_width} ${prism_width} ${sqrt_2*base_z}"/>
             </geometry>
-            <origin xyz="${-0.4/2} 0 ${-0.4/2}" rpy="0 ${pi/4} 0"/>
+            <origin xyz="${-axle_height/2} 0 ${-axle_height/2}" rpy="0 ${pi/4} 0"/>
         </visual>
         <visual>
             <geometry>
-                <box size="0.05 0.05 ${sqrt_2*0.4}"/>
+                <box size="${prism_width} ${prism_width} ${sqrt_2*base_z}"/>
             </geometry>
-            <origin xyz="${0.4/2} 0 ${-0.4/2}" rpy="0 ${-pi/4} 0"/>
+            <origin xyz="${axle_height/2} 0 ${-axle_height/2}" rpy="0 ${-pi/4} 0"/>
         </visual>
         <collision>
             <geometry>
-                <box size="0.05 0.05 ${sqrt_2*0.4}"/>
+                <box size="${prism_width} ${prism_width} ${sqrt_2*base_z}"/>
             </geometry>
-            <origin xyz="${-0.4/2} 0 ${-0.4/2}" rpy="0 ${pi/4} 0"/>
+            <origin xyz="${-axle_height/2} 0 ${-axle_height/2}" rpy="0 ${pi/4} 0"/>
         </collision>
         <collision>
             <geometry>
-                <box size="0.05 0.05 ${sqrt_2*0.4}"/>
+                <box size="${prism_width} ${prism_width} ${sqrt_2*base_z}"/>
             </geometry>
-            <origin xyz="${0.4/2} 0 ${-0.4/2}" rpy="0 ${-pi/4} 0"/>
+            <origin xyz="${axle_height/2} 0 ${-axle_height/2}" rpy="0 ${-pi/4} 0"/>
         </collision>
         <inertial>
@@ -153,5 +165,5 @@
         <parent link="base_link"/>
         <child link="rear_axle_link"/>
-        <origin xyz="${-1/2} 0 -0.15" rpy="0 0 0"/>
+        <origin xyz="${-base_x/2} 0 -0.15" rpy="0 0 0"/>
         <axis xyz="1 0 0"/>
     </joint>
@@ -159,5 +171,5 @@
         <parent link="base_link"/>
         <child link="front_left_axle_link"/>
-        <origin xyz="0.3 ${0.3+0.05/2} -0.15" rpy="0 0 0"/>
+        <origin xyz="0.3 ${0.3+prism_width/2} -0.15" rpy="0 0 0"/>
         <axis xyz="0 1 0"/>
     </joint>
@@ -165,20 +177,17 @@
         <parent link="base_link"/>
         <child link="front_right_axle_link"/>
-        <origin xyz="0.3 ${-(0.3+0.05/2)} -0.15" rpy="0 0 0"/>
+        <origin xyz="0.3 ${-(0.3+prism_width/2)} -0.15" rpy="0 0 0"/>
         <axis xyz="0 1 0"/>
     </joint>
-    <!--
-        <xacro:wheel prefix="" parent="" x="${}" y="${}" z="${}" roll="${}"/>
-    -->
-    <xacro:wheel prefix="back_left_wheel" parent="rear_axle_link" x="${-0.05-0.05/2}" y="${0.6/2+0.05+0.1/2}" z="-0.4" roll="${pi/2}"/>
-    <xacro:wheel prefix="back_right_wheel" parent="rear_axle_link" x="${-0.05-0.05/2}" y="${-(0.6/2+0.05+0.1/2)}" z="-0.4" roll="${-pi/2}"/>
-    <xacro:wheel prefix="center_left_wheel" parent="front_left_axle_link" x="${-0.4}" y="${0.05/2+0.1/2}" z="${-0.4}" roll="${pi/2}"/>
-    <xacro:wheel prefix="center_right_wheel" parent="front_right_axle_link" x="${-0.4}" y="${-(0.05/2+0.1/2)}" z="${-0.4}" roll="${-pi/2}"/>
-    <xacro:wheel prefix="front_left_wheel" parent="front_left_axle_link" x="${0.4}" y="${0.05/2+0.1/2}" z="${-0.4}" roll="${pi/2}"/>
-    <xacro:wheel prefix="front_right_wheel" parent="front_right_axle_link" x="${0.4}" y="${-(0.05/2+0.1/2)}" z="${-0.4}" roll="${-pi/2}"/>
+    <xacro:wheel prefix="back_left_wheel" parent="rear_axle_link" x="${-rear_cyl_l-prism_width/2}" y="${rear_width/2+prism_width+0.1/2}" z="${-axle_height}" width="${wheel_width}" radius="${wheel_radius}" roll="${pi/2}"/>
+    <xacro:wheel prefix="back_right_wheel" parent="rear_axle_link" x="${-rear_cyl_l-prism_width/2}" y="${-(rear_width/2+prism_width+0.1/2)}" z="${-axle_height}" width="${wheel_width}" radius="${wheel_radius}" roll="${-pi/2}"/>
+    <xacro:wheel prefix="center_left_wheel" parent="front_left_axle_link" x="${-axle_height}" y="${prism_width/2+0.1/2}" z="${-axle_height}" width="${wheel_width}" radius="${wheel_radius}" roll="${pi/2}"/>
+    <xacro:wheel prefix="center_right_wheel" parent="front_right_axle_link" x="${-axle_height}" y="${-(prism_width/2+0.1/2)}" z="${-axle_height}" width="${wheel_width}" radius="${wheel_radius}" roll="${-pi/2}"/>
+    <xacro:wheel prefix="front_left_wheel" parent="front_left_axle_link" x="${axle_height}" y="${prism_width/2+0.1/2}" z="${-axle_height}" width="${wheel_width}" radius="${wheel_radius}" roll="${pi/2}"/>
+    <xacro:wheel prefix="front_right_wheel" parent="front_right_axle_link" x="${axle_height}" y="${-(prism_width/2+0.1/2)}" z="${-axle_height}" width="${wheel_width}" radius="${wheel_radius}" roll="${-pi/2}"/>
 </robot>
 <!--
 EJECUTAR ESTA LINEA ANTES DE HACER catkin_make
 rosrun xacro xacro ~/catkin_ws/src/donatello_sim/urdf/donatello.urdf.xacro > ~/catkin_ws/src/donatello_sim/urdf/donatello.urdf
-check_urdf ~/catkin_ws/donatello_sim/urdf/donatello.urdf
+check_urdf ~/catkin_ws/src/donatello_sim/urdf/donatello.urdf
 -->

File: urdf/donatello_include.xacro (robot description, xacro)
@@ -1,9 +1,9 @@
 <?xml version="1.0"?>
 <robot xmlns:xacro="http://www.ros.org/wiki/xacro">
-<xacro:macro name="wheel" params="prefix parent x y z roll">
+<xacro:macro name="wheel" params="prefix parent x y z width radius roll">
     <link name="${prefix}_link">
         <visual>
             <geometry>
-                <cylinder length="0.1" radius="0.1"/>
+                <cylinder length="${width}" radius="${radius}"/>
             </geometry>
             <origin xyz="0 0 0" rpy="0 0 0"/>
@@ -11,5 +11,5 @@
         <collision>
             <geometry>
-                <cylinder length="0.1" radius="0.1"/>
+                <cylinder length="${width}" radius="${radius}"/>
             </geometry>
             <origin xyz="0 0 0" rpy="0 0 0"/>

Commit message: 24/10/24. Medición y inicio en urdf

File: urdf/donatello.urdf (robot description, URDF)
Before this commit: robot donatello, 11 links, 10 joints
Links:
- link base_link: geometry collision box size=5.0 3.48 1.65; visual box size=5.0 3.48 1.65
- link rear_axle_link: geometry collision box size=0.05 0.05 0.4; collision box size=0.05 0.05 0.4

Commit message: DisTriangulo+MovimientoPiezas

File: urdf/donatello.urdf (robot description, URDF)
Before this commit: robot donatello, 11 links, 10 joints
Links:
- link front_left_axle_link: geometry collision box size=0.3 0.3 2.6; collision box size=0.3 0.3 2.6
- link front_right_axle_link: geometry collision box size=0.3 0.3 2.6; collision box size=0.3 0.3 2.6

Commit message: ActuURDF

File: urdf/donatello.urdf (robot description, URDF)
Before this commit: robot donatello, 11 links, 10 joints
Links:
- link rear_axle_link: geometry collision box size=0.05 0.05 0.4; collision box size=0.05 0.05 0.4

Commit message: Paso_a_metros_medio_posicionado

File: urdf/donatello.urdf (robot description, URDF)
Before this commit: robot donatello, 11 links, 10 joints
Links:
- link back_left_wheel_link: geometry collision cylinder length=0.07 radius=0.045; visual cylinder length=0.07 radius=0.045
- link back_right_wheel_link: geometry collision cylinder length=0.07 radius=0.045; visual cylinder length=0.07 radius=0.045
- link base_link: geometry collision box size=0.55 0.35 0.165; visual box size=0.55 0.35 0.165
- link center_left_wheel_link: geometry collision cylinder length=0.07 radius=0.045; visual cylinder length=0.07 radius=0.045
- link center_right_wheel_link: geometry collision cylinder length=0.07 radius=0.045; visual cylinder length=0.07 radius=0.045
- link front_left_axle_link: geometry collision box size=0.03 0.03 0.26; collision box size=0.03 0.03 0.26
- link front_left_wheel_link: geometry collision cylinder length=0.07 radius=0.045; visual cylinder length=0.07 radius=0.045
- link front_right_axle_link: geometry collision box size=0.03 0.03 0.26; collision box size=0.03 0.03 0.26
- link front_right_wheel_link: geometry collision cylinder length=0.07 radius=0.045; visual cylinder length=0.07 radius=0.045
- link rear_axle_link: geometry collision box size=0.05 0.05 0.4; collision box size=0.05 0.05 0.4
Joints:
- joint front_left_wheel_joint: origin xyz=0.4 0.07500000000000001 -0.4 rpy=1.5707963 0 0 -> xyz=0 0 0 rpy=1.5707963 0 0

Commit message: Update_medidas

File: urdf/donatello.urdf (robot description, URDF)
Before this commit: robot donatello, 11 links, 10 joints
Links:
- link front_left_axle_link: geometry collision box size=0.03 0.03 0.26; collision box size=0.03 0.03 0.26
- link front_right_axle_link: geometry collision box size=0.03 0.03 0.23; collision box size=0.03 0.03 0.26
